File: hardware/jaja.kicad_pcb (KiCad board)
At the start: 2 copper layers, 124 parts, among them SW1 SW_SPST, SW10 SW_SPST, SW11 SW_SPST, SW12 SW_SPST, SW13 SW_SPST, SW14 SW_SPST, SW15 SW_SPST, SW16 SW_SPST, SW17 SW_SPST, SW18 SW_SPST, SW19 SW_SPST, SW2 SW_SPST, SW20 SW_SPST, SW21 SW_SPST, SW22 SW_SPST, SW23 SW_SPST, SW24 SW_SPST, SW25 SW_SPST, SW26 SW_SPST, SW27 SW_SPST, SW28 SW_SPST, SW29 SW_SPST, SW3 SW_SPST, SW30 SW_SPST, SW31 SW_SPST, SW32 SW_SPST, SW33 SW_SPST, SW34 SW_SPST, SW35 SW_SPST, SW36 SW_SPST, SW37 SW_SPST, SW38 SW_SPST, SW39 SW_SPST, SW4 SW_SPST, SW40 SW_SPST, SW41 SW_SPST, SW42 SW_SPST, SW43 SW_SPST, SW44 SW_SPST, SW45 SW_SPST, SW46 SW_SPST, SW47 SW_SPST, SW48 SW_SPST, SW49 SW_SPST, SW5 SW_SPST, SW50 SW_SPST, SW51 SW_SPST, SW52 SW_SPST, SW53 SW_SPST, SW54 SW_SPST, SW55 SW_SPST, SW56 SW_SPST, SW57 SW_SPST, SW58 SW_SPST, SW59 SW_SPST, SW6 SW_SPST, SW60 SW_SPST, SW61 SW_SPST, SW7 SW_SPST, SW8 SW_SPST, SW9 SW_SPST

Commit message: Add LED library
Parts:
- added D62: SK6812MINI, Keebio-Parts:SK6812-MINI-E, F.Cu at (63.5, 35.6)
- moved D2 7.63 mm to (69.5, 35.6)
Other:
- board outline added: 337.9 x 137.3 mm
Changed lines of the file:
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@@
   (net 82 "unconnected-(LED1-VSS-Pad3)")
   (net 83 "unconnected-(LED1-DIN-Pad4)")
+  (net 84 "unconnected-(D62-DOUT-Pad1)")
+  (net 85 "unconnected-(D62-VSS-Pad2)")
+  (net 86 "unconnected-(D62-VDD-Pad4)")
+  (net 87 "unconnected-(D62-DIN-Pad3)")
   (footprint "PCM_Mounting_Keyboard_Stabilizer:Stabilizer_Cherry_MX_6.25u" (layer "F.Cu")
     (at 208.28 137.16)
@@
   )
   (footprint "Diode_SMD:D_SOD-123" (layer "F.Cu")
-    (at 62.865 31.75)
+    (at 69.47 35.56)
     (descr "SOD-123")
     (tags "SOD-123")
@@
     )
   )
+  (footprint "Keebio-Parts:SK6812-MINI-E" (layer "F.Cu")
+    (at 63.5 35.56)
+    (property "Sheetfile" "jaja.kicad_sch")
+    (property "Sheetname" "")
+    (property "ki_description" "RGB LED with integrated controller")
+    (property "ki_keywords" "RGB LED NeoPixel Mini addressable")
+    (attr through_hole)
+    (fp_text reference "D62" (at 0 2.1 unlocked) (layer "F.SilkS")
+        (effects (font (size 0.7 0.7) (thickness 0.15)))
+    )
+    (fp_text value "SK6812MINI" (at 0 -0.5 unlocked) (layer "F.SilkS") hide
+        (effects (font (size 1 1) (thickness 0.15)))
+    )
+    (fp_poly
+      (pts
+        (xy 2.8 -1.4)
+        (xy 2.2 -1.4)
+        (xy 2.2 -2)
+      )
+      (stroke (width 0.1) (type solid)) (fill solid) (layer "F.SilkS"))
+    (fp_line (start -1.6 -1.4) (end 1.6 -1.4)
+      (stroke (width 0.12) (type solid)) (layer "Cmts.User"))
+    (fp_line (start -1.6 1.4) (end -1.6 -1.4)
+      (stroke (width 0.12) (type solid)) (layer "Cmts.User"))
+    (fp_line (start 1.6 -1.4) (end 1.6 1.4)
+      (stroke (width 0.12) (type solid)) (layer "Cmts.User"))
+    (fp_line (start 1.6 1.4) (end -1.6 1.4)
+      (stroke (width 0.12) (type solid)) (layer "Cmts.User"))
+    (fp_line (start -1.7 -1.5) (end 1.7 -1.5)
+      (stroke (width 0.12) (type solid)) (layer "Edge.Cuts"))
+    (fp_line (start -1.7 1.5) (end -1.7 -1.5)
+      (stroke (width 0.12) (type solid)) (layer "Edge.Cuts"))
+    (fp_line (start 1.7 -1.5) (end 1.7 1.5)
+      (stroke (width 0.12) (type solid)) (layer "Edge.Cuts"))
+    (fp_line (start 1.7 1.5) (end -1.7 1.5)
+      (stroke (width 0.12) (type solid)) (layer "Edge.Cuts"))
+    (pad "1" smd rect (at -2.55 0.75) (size 1.7 0.82) (layers "F.Cu" "F.Paste" "F.Mask")
+      (net 84 "unconnected-(D62-DOUT-Pad1)") (pinfunction "DOUT") (pintype "output"))
+    (pad "2" smd rect (at -2.55 -0.75) (size 1.7 0.82) (layers "F.Cu" "F.Paste" "F.Mask")
+      (net 85 "unconnected-(D62-VSS-Pad2)") (pinfunction "VSS") (pintype "power_in"))
+    (pad "3" smd roundrect (at 2.55 -0.75) (size 1.7 0.82) (layers "F.Cu" "F.Paste" "F.Mask") (roundrect_rratio 0.25)
+      (net 87 "unconnected-(D62-DIN-Pad3)") (pinfunction "DIN") (pintype "input"))
+    (pad "4" smd rect (at 2.55 0.75) (size 1.7 0.82) (layers "F.Cu" "F.Paste" "F.Mask")
+      (net 86 "unconnected-(D62-VDD-Pad4)") (pinfunction "VDD") (pintype "power_in"))
+    (model "/Users/danny/syncproj/kicad-libs/footprints/Keebio-Parts.pretty/3dmodels/SK6812MINI-E v1.step"
+      (offset (xyz 0 0 0))
+      (scale (xyz 1 1 1))
+      (rotate (xyz 90 0 0))
+    )
+  )
   (footprint "Diode_SMD:D_SOD-123" (layer "F.Cu")
     (at 77.1525 69.85)
@@
     )
   )
+  (gr_poly
+    (pts
+      (xy 360.68 15.19)
+      (xy 360.715355 15.204645)
+      (xy 360.73 15.24)
+      (xy 360.73 152.4)
+      (xy 360.715355 152.435355)
+      (xy 360.68 152.45)
+      (xy 22.86 152.45)
+      (xy 22.824645 152.435355)
+      (xy 22.81 152.4)
+      (xy 22.81 15.24)
+      (xy 22.824645 15.204645)
+      (xy 22.86 15.19)
+    )
+    (stroke (width 0.1) (type solid)) (fill none) (layer "Edge.Cuts"))
 )
