File: hardware/jaja.kicad_sch (KiCad schematic)
At the start: 123 parts, among them SW1 SW_SPST, SW10 SW_SPST, SW11 SW_SPST, SW12 SW_SPST, SW13 SW_SPST, SW14 SW_SPST, SW15 SW_SPST, SW16 SW_SPST, SW17 SW_SPST, SW18 SW_SPST, SW19 SW_SPST, SW2 SW_SPST, SW20 SW_SPST, SW21 SW_SPST, SW22 SW_SPST, SW23 SW_SPST, SW24 SW_SPST, SW25 SW_SPST, SW26 SW_SPST, SW27 SW_SPST, SW28 SW_SPST, SW29 SW_SPST, SW3 SW_SPST, SW30 SW_SPST, SW31 SW_SPST, SW32 SW_SPST, SW33 SW_SPST, SW34 SW_SPST, SW35 SW_SPST, SW36 SW_SPST, SW37 SW_SPST, SW38 SW_SPST, SW39 SW_SPST, SW4 SW_SPST, SW40 SW_SPST, SW41 SW_SPST, SW42 SW_SPST, SW43 SW_SPST, SW44 SW_SPST, SW45 SW_SPST, SW46 SW_SPST, SW47 SW_SPST, SW48 SW_SPST, SW49 SW_SPST, SW5 SW_SPST, SW50 SW_SPST, SW51 SW_SPST, SW52 SW_SPST, SW53 SW_SPST, SW54 SW_SPST, SW55 SW_SPST, SW56 SW_SPST, SW57 SW_SPST, SW58 SW_SPST, SW59 SW_SPST, SW6 SW_SPST, SW60 SW_SPST, SW61 SW_SPST, SW7 SW_SPST, SW8 SW_SPST, SW9 SW_SPST

Commit message: Add LED library
Parts:
- added D62: SK6812MINI, Keebio-Parts:SK6812-MINI-E, symbol LED:SK6812MINI
Changed lines of the file:
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@@
+    )
+  )
+  (symbol (lib_id "LED:SK6812MINI") (at 148.59 160.02 0) (unit 1)
+    (in_bom yes) (on_board yes) (dnp no) (fields_autoplaced)
+    (property "Reference" "D62" (at 161.29 156.8959 0)
+      (effects (font (size 1.27 1.27)))
+    )
+    (property "Value" "SK6812MINI" (at 161.29 159.4359 0)
+      (effects (font (size 1.27 1.27)))
+    )
+    (property "Footprint" "Keebio-Parts:SK6812-MINI-E" (at 149.86 167.64 0)
+      (effects (font (size 1.27 1.27)) (justify left top) hide)
+    )
+    (property "Datasheet" "https://cdn-shop.adafruit.com/product-files/2686/SK6812MINI_REV.01-1-2.pdf" (at 151.13 169.545 0)
+      (effects (font (size 1.27 1.27)) (justify left top) hide)
+    )
+    (pin "1")
+    (pin "2")
+    (pin "3")
+    (pin "4")
+    (instances
+      (project "jaja"
+        (path "/5d1842fd-b488-4aaf-9554-5dd11731426c"
+          (reference "D62") (unit 1)
+        )
+      )
     )
   )
